File: fluidnc-bob.kicad_pcb (KiCad board)
At the start: 2 copper layers, 157.5 x 96.5 mm, 44 parts, among them J1 X_Limit, J10 Z_stepdir, J11 spindle_pwm_dir, J12 Flood_Mist, J13 GND, J14 GND, J15 +5v, J16 +5v, J2 Y_Limit, J3 Hold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

Commit message: Add files via upload
Other:
- board text added: "5V"
- board text added: "EXT 5V INPUT"
- board text added: "EXT GND INPUT"
- board text added: "GND"
Changed lines of the file:
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@@
     (effects (font (size 1 1) (thickness 0.15)))
+  )
+  (gr_text "EXT GND\nINPUT" (at 100.076 51.562) (layer "F.SilkS")
+    (effects (font (size 1 1) (thickness 0.15)) (justify left bottom))
   )
   (gr_text "Probe" (at 64.77 111.76) (layer "F.SilkS")
@@
   (gr_text "FluidNC\nBreak-Out Board v1.0" (at 165.1 116.84) (layer "F.SilkS")
     (effects (font (size 1 1) (thickness 0.15)))
+  )
+  (gr_text "GND" (at 114.046 50.546) (layer "F.SilkS")
+    (effects (font (size 1 1) (thickness 0.15)) (justify left bottom))
   )
   (gr_text "STEP" (at 214.63 86.36) (layer "F.SilkS")
@@
     (effects (font (size 1 1) (thickness 0.15)))
   )
+  (gr_text "5V" (at 127.762 50.292) (layer "F.SilkS")
+    (effects (font (size 1 1) (thickness 0.15)) (justify left bottom))
+  )
   (gr_text "X-axis" (at 214.63 83.82) (layer "F.SilkS")
     (effects (font (size 1 1) (thickness 0.15)))
@@
     (effects (font (size 1 1) (thickness 0.15)))
   )
+  (gr_text "EXT 5V \nINPUT" (at 138.43 51.308) (layer "F.SilkS")
+    (effects (font (size 1 1) (thickness 0.15)) (justify left bottom))
+  )
   (gr_text "STEP" (at 214.63 99.06) (layer "F.SilkS")

Commit message: Add files via upload
Other:
- board text added: "EXT 5V (Mandatory)"
- board text removed: "EXT 5V INPUT"
- board text removed: "EXT GND INPUT"
Changed lines of the file:
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@@
     (tags "THT terminal block Metz Connect Type073_RT02602HBLU pitch 5.08mm size 10.2x11mm^2 drill 1.4mm pad 2.6mm")
     (attr through_hole)
-    (fp_text reference "J1" (at 2.54 -6.56 90) (layer "F.SilkS")
+    (fp_text reference "J1" (at 2.54 7.62 90) (layer "F.SilkS")
         (effects (font (size 1 1) (thickness 0.15)))
     )
@@
     (tags "THT terminal block Metz Connect Type073_RT02602HBLU pitch 5.08mm size 10.2x11mm^2 drill 1.4mm pad 2.6mm")
     (attr through_hole)
-    (fp_text reference "J2" (at 2.54 -6.56 90) (layer "F.SilkS")
+    (fp_text reference "J2" (at 2.54 7.62 90) (layer "F.SilkS")
         (effects (font (size 1 1) (thickness 0.15)))
     )
@@
     (tags "THT terminal block Metz Connect Type073_RT02602HBLU pitch 5.08mm size 10.2x11mm^2 drill 1.4mm pad 2.6mm")
     (attr through_hole)
-    (fp_text reference "J3" (at 2.54 -6.56 90) (layer "F.SilkS")
+    (fp_text reference "J3" (at 2.54 7.874 90) (layer "F.SilkS")
         (effects (font (size 1 1) (thickness 0.15)))
     )
@@
     (tags "THT terminal block Metz Connect Type073_RT02602HBLU pitch 5.08mm size 10.2x11mm^2 drill 1.4mm pad 2.6mm")
     (attr through_hole)
-    (fp_text reference "J4" (at 2.54 -6.56 90) (layer "F.SilkS")
+    (fp_text reference "J4" (at 2.54 7.62 90) (layer "F.SilkS")
         (effects (font (size 1 1) (thickness 0.15)))
     )
@@
     (tags "THT terminal block Metz Connect Type073_RT02602HBLU pitch 5.08mm size 10.2x11mm^2 drill 1.4mm pad 2.6mm")
     (attr through_hole)
-    (fp_text reference "J5" (at 2.54 -6.56 90) (layer "F.SilkS")
+    (fp_text reference "J5" (at 2.286 7.874 90) (layer "F.SilkS")
         (effects (font (size 1 1) (thickness 0.15)))
     )
@@
     (tags "THT terminal block Metz Connect Type073_RT02602HBLU pitch 5.08mm size 10.2x11mm^2 drill 1.4mm pad 2.6mm")
     (attr through_hole)
-    (fp_text reference "J6" (at 2.54 -6.56 90) (layer "F.SilkS")
+    (fp_text reference "J6" (at 2.286 7.62 90) (layer "F.SilkS")
         (effects (font (size 1 1) (thickness 0.15)))
     )
@@
     (tags "THT terminal block Metz Connect Type073_RT02602HBLU pitch 5.08mm size 10.2x11mm^2 drill 1.4mm pad 2.6mm")
     (attr through_hole)
-    (fp_text reference "J7" (at 2.54 -6.56 90) (layer "F.SilkS")
+    (fp_text reference "J7" (at 2.54 7.62 90) (layer "F.SilkS")
         (effects (font (size 1 1) (thickness 0.15)))
     )
@@
     (tags "THT terminal block Metz Connect Type073_RT02602HBLU pitch 5.08mm size 10.2x11mm^2 drill 1.4mm pad 2.6mm")
     (attr through_hole)
-    (fp_text reference "J8" (at 2.54 -6.56 90) (layer "F.SilkS")
+    (fp_text reference "J8" (at 2.286 7.62 90) (layer "F.SilkS")
         (effects (font (size 1 1) (thickness 0.15)))
     )
@@
     (tags "THT terminal block Metz Connect Type073_RT02602HBLU pitch 5.08mm size 10.2x11mm^2 drill 1.4mm pad 2.6mm")
     (attr through_hole)
-    (fp_text reference "J9" (at 2.54 -6.56 90) (layer "F.SilkS")
+    (fp_text reference "J9" (at 2.286 7.62 90) (layer "F.SilkS")
         (effects (font (size 1 1) (thickness 0.15)))
     )
@@
     (tags "THT terminal block Metz Connect Type073_RT02602HBLU pitch 5.08mm size 10.2x11mm^2 drill 1.4mm pad 2.6mm")
     (attr through_hole)
-    (fp_text reference "J10" (at 2.54 -6.56 90) (layer "F.SilkS")
+    (fp_text reference "J10" (at 2.286 7.62 90) (layer "F.SilkS")
         (effects (font (size 1 1) (thickness 0.15)))
     )
@@
     (tags "THT terminal block Metz Connect Type073_RT02602HBLU pitch 5.08mm size 10.2x11mm^2 drill 1.4mm pad 2.6mm")
     (attr through_hole)
-    (fp_text reference "J11" (at 2.54 -6.56 90) (layer "F.SilkS")
+    (fp_text reference "J11" (at 2.54 7.366 90) (layer "F.SilkS")
         (effects (font (size 1 1) (thickness 0.15)))
     )
@@
     (tags "THT terminal block Metz Connect Type073_RT02602HBLU pitch 5.08mm size 10.2x11mm^2 drill 1.4mm pad 2.6mm")
     (attr through_hole)
-    (fp_text reference "J12" (at 2.54 -6.56 90) (layer "F.SilkS")
+    (fp_text reference "J12" (at 2.54 7.62 90) (layer "F.SilkS")
         (effects (font (size 1 1) (thickness 0.15)))
     )
@@
     (effects (font (size 1 1) (thickness 0.15)))
   )
-  (gr_text "Limit\nX\n" (at 64.77 48.26) (layer "F.SilkS")
+  (gr_text "Limit\nX\n" (at 64.77 51.054) (layer "F.SilkS")
     (effects (font (size 1 1) (thickness 0.15)))
   )
-  (gr_text "EXT GND\nINPUT" (at 100.076 51.562) (layer "F.SilkS")
+  (gr_text "GND" (at 101.346 50.546) (layer "F.SilkS")
     (effects (font (size 1 1) (thickness 0.15)) (justify left bottom))
   )
-  (gr_text "Probe" (at 64.77 111.76) (layer "F.SilkS")
+  (gr_text "Probe" (at 64.77 114.3) (layer "F.SilkS")
     (effects (font (size 1 1) (thickness 0.15)))
   )
-  (gr_text "Door" (at 64.77 86.36) (layer "F.SilkS")
+  (gr_text "Door" (at 64.77 88.9) (layer "F.SilkS")
     (effects (font (size 1 1) (thickness 0.15)))
   )
@@
     (effects (font (size 1 1) (thickness 0.15)))
   )
-  (gr_text "Hold" (at 64.77 99.06) (layer "F.SilkS")
+  (gr_text "Hold" (at 64.77 101.346) (layer "F.SilkS")
     (effects (font (size 1 1) (thickness 0.15)))
   )
-  (gr_text "Limit \nY" (at 64.77 60.96) (layer "F.SilkS")
+  (gr_text "Limit \nY" (at 64.77 63.5) (layer "F.SilkS")
     (effects (font (size 1 1) (thickness 0.15)))
   )
-  (gr_text "Limit\nZ" (at 64.77 73.66) (layer "F.SilkS")
+  (gr_text "Limit\nZ" (at 64.77 76.2) (layer "F.SilkS")
     (effects (font (size 1 1) (thickness 0.15)))
   )
@@
     (effects (font (size 1 1) (thickness 0.15)))
   )
-  (gr_text "5V" (at 127.762 50.292) (layer "F.SilkS")
+  (gr_text "5V" (at 128.016 50.546) (layer "F.SilkS")
     (effects (font (size 1 1) (thickness 0.15)) (justify left bottom))
   )
@@
     (effects (font (size 1 1) (thickness 0.15)))
   )
-  (gr_text "EXT 5V \nINPUT" (at 138.43 51.308) (layer "F.SilkS")
-    (effects (font (size 1 1) (thickness 0.15)) (justify left bottom))
+  (gr_text "EXT 5V\n(Mandatory)\n" (at 140.97 51.308) (layer "F.SilkS")
+    (effects (font (size 1 1) (thickness 0.15)) (justify bottom))
   )
   (gr_text "STEP" (at 214.63 99.06) (layer "F.SilkS")
